Commit message: 20220420

File: portaal_robot/portaal_robot_description/urdf/portaal_robot.urdf.xacro (robot description, xacro)
@@ -2,4 +2,19 @@
 <!-- portaal_robot Chain -->
 <robot name="portaal_robot" xmlns:xacro="http://ros.org/wiki/xacro">
+  <xacro:macro name="cylinder_inertia" params="m r h">
+        <inertia  ixx="${m*(3*r*r+h*h)/12}" ixy = "0" ixz = "0"
+                    iyy="${m*(3*r*r+h*h)/12}" iyz = "0"
+                    izz="${m*r*r/2}" />
+  </xacro:macro>
+  <xacro:macro name="box_inertia" params="m x y z">
+          <inertia  ixx="${m*(y*y+z*z)/12}" ixy = "0" ixz = "0"
+                    iyy="${m*(x*x+z*z)/12}" iyz = "0"
+                    izz="${m*(x*x+z*z)/12}" />
+  </xacro:macro>
+  <xacro:macro name="sphere_inertia" params="m r">
+          <inertia  ixx="${2*m*r*r/5}" ixy = "0" ixz = "0"
+                    iyy="${2*m*r*r/5}" iyz = "0"
+                    izz="${2*m*r*r/5}" />
+  </xacro:macro>
   <material name="LightGrey">
       <color rgba="0.7 0.7 0.7 1.0" />
@@ -21,8 +36,6 @@
     <inertial>
       <origin xyz="0 0 0" rpy="0 0 0" />
-      <inertia ixx="0.1" ixy="0" ixz="0"
-               iyy="0.1" iyz="0"
-               izz="0.1" />
-      <mass value="1" />
+      <mass value="1"/>
+      <xacro:box_inertia m="1" x="0.04" y="1.5" z="0.04"/>
     </inertial>
     <visual>
@@ -37,8 +50,6 @@
     <inertial>
       <origin xyz="0 0 0" rpy="0 0 0" />
-      <inertia ixx="0.1" ixy="0" ixz="0"
-               iyy="0.1" iyz="0"
-               izz="0.1" />
-      <mass value="1" />
+      <mass value="0.1"/>
+      <xacro:box_inertia m="0.1" x="0.04" y="0.04" z="0.04"/>
     </inertial>
     <visual>
@@ -67,8 +78,6 @@
     <inertial>
       <origin xyz="0 0 0" rpy="0 0 0" />
-      <inertia ixx="0.1" ixy="0" ixz="0"
-               iyy="0.1" iyz="0"
-               izz="0.1" />
-      <mass value="1" />
+      <mass value="0.75"/>
+      <xacro:box_inertia m="0.75" x="0.043" y="0.03" z="1.0"/>
     </inertial>
     <visual>
@@ -92,4 +101,9 @@
   </joint>
   <link name="vacuum_gripper">
+    <inertial>
+      <origin xyz="0 0 0" rpy="0 0 0" />
+      <mass value="1"/>
+      <xacro:cylinder_inertia m="1" r="1.5" h="0.015"/>
+    </inertial>
     <visual>
       <origin xyz="0 0 0" />
